File: fabrication/Switchboard/CD40106_VCO.kicad_pcb (KiCad board)
At the start: 2 copper layers, 28 x 38.5 mm, 7 parts, among them J12 Conn_01x04, SW1 Octave select switch

Commit message: V2.0
Parts:
- moved R25 96.2 mm to (41.6, 65.0)
- moved J12 96.2 mm to (40.5, 72.2)
- moved R20 96.2 mm to (16.4, 65.0)
- moved R22 96.2 mm to (16.4, 68.2)
- moved R23 96.2 mm to (26.6, 71.5)
- moved R26 96.2 mm to (31.4, 68.2)
- moved SW1 96.2 mm to (29.0, 50.0)
Other:
- board text added: "1"
- board text added: "2"
- board text added: "3"
- board text added: "4"
- board text added: "Board 3"
- board text added: "CD40106 VCO 2.0 Bleep Sound 2025"
