File: fabrication/circuitboard/CD40106_VCO.kicad_pcb (KiCad board)
At the start: 2 copper layers, 50 x 110 mm, 87 parts, among them J11 Conn_01x04, J14 Conn_01x02, J16 Power Input, J5 Conn_Circuit, J7 Conn_Circuit, Q1 BC558, Q2 BC548, U1 TL074, U2 CD40106, U3 LM336BZ-5.0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

Commit message: V2.0
Parts:
- removed C1: 2.2nF, Kicad-perso:Mica Disc Cap
- removed FB1, FB2: 10R, Inductor_THT:L_Axial_L7.0mm_D3.3mm_P10.16mm_Horizontal_Fastron_MICC
- added C23: 2.2nF, Capacitor_THT:C_Disc_D7.0mm_W2.5mm_P5.00mm, F.Cu at (102.3, 130.2)
- added D1: 1N4148, Diode_THT:D_DO-35_SOD27_P7.62mm_Horizontal, F.Cu at (75.5, 84.8)
- added D6: 1N5819, Diode_THT:D_DO-41_SOD81_P10.16mm_Horizontal, F.Cu at (92.8, 134.9)
- added D8: 1N5819, Diode_THT:D_DO-41_SOD81_P10.16mm_Horizontal, F.Cu at (66.7, 145.1)
- added Q3: BC548, Package_TO_SOT_THT:TO-92_Inline, F.Cu at (75.8, 80.6)
- added Q4: BC558, Package_TO_SOT_THT:TO-92_Inline, F.Cu at (81.3, 80.6)
- added R43: 20k, Resistor_THT:R_Axial_DIN0207_L6.3mm_D2.5mm_P10.16mm_Horizontal, F.Cu at (78.5, 116.9)
- added R45: 20k, Resistor_THT:R_Axial_DIN0207_L6.3mm_D2.5mm_P10.16mm_Horizontal, F.Cu at (74.6, 132.0)
- added R46: 47k, Resistor_THT:R_Axial_DIN0207_L6.3mm_D2.5mm_P10.16mm_Horizontal, F.Cu at (72.7, 82.2)
- added R47: 2.2k, Resistor_THT:R_Axial_DIN0207_L6.3mm_D2.5mm_P10.16mm_Horizontal, F.Cu at (85.6, 73.2)
- added R48: 10k, Resistor_THT:R_Axial_DIN0207_L6.3mm_D2.5mm_P10.16mm_Horizontal, F.Cu at (85.6, 76.3)
- C13, C18, C19, C4, C5, C7, R16, R17, R18, R19, R21, U4: moved to B.Cu
- C2: value Optionnal -> 2.2nF; footprint Capacitor_THT:C_Disc_D7.0mm_W2.5mm_P5.00mm -> Capacitor_THT:C_Rect_L7.0mm_W2.5mm_P5.00mm
- R13: value 1M -> 100k
- R24: value 9k53 -> 9k1; moved to B.Cu
- R29: value 20k -> 1k
- R30, R39: value 200k -> 330k
- R40: value 10k -> 33k
- R42: value 10k -> 100k
- Sine_Bias_trim1, Sine_Lvl_trim1, Sine_Shape_trim1, lvl_Trim1: footprint Potentiometer_THT:Potentiometer_Bourns_3386C_Horizontal -> Potentiometer_THT:Potentiometer_Bourns_3296W_Vertical
- U3: value LM336BZ-5.0 -> LM336-2.5; moved to B.Cu
- lvl_Trim2: value 1k -> 2k; footprint Potentiometer_THT:Potentiometer_Bourns_3386C_Horizontal -> Potentiometer_THT:Potentiometer_Bourns_3296W_Vertical
- moved C7 23.6 mm to (80.0, 61.3), turned to 180 degrees
- moved TP3 20.8 mm to (57.2, 53.8)
- moved C19 14.1 mm to (75.2, 58.5)
- moved C18 14.0 mm to (61.2, 61.3)
- moved TP2 10.7 mm to (87.3, 80.4)
- moved U4 7.60 mm to (64.4, 53.7)
- moved TH3 6.65 mm to (71.9, 76.0), turned to -90 degrees
- moved D2 5.60 mm to (78.1, 84.8)
- moved J11 5.07 mm to (96.0, 73.1), turned to 180 degrees
- moved C4 5.00 mm to (68.5, 67.7), turned to 0 degrees
- moved C17 4.97 mm to (72.7, 128.8), turned to 180 degrees
- moved U1 3.70 mm to (75.3, 118.1)
- moved U3 2.54 mm to (76.3, 68.2), turned to 0 degrees
- moved C2 1.60 mm to (80.9, 92.2)
- moved R44 1.10 mm to (99.1, 138.5)
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Connections:
- C2 pad 1: /Sync -> Net-(D2-K)
- C8 pad 1: /Saw -> Net-(C8-Pad1)
- D2 pad 1: /Sync -> Net-(D2-K)
- Q1 pad 1: Net-(Q1-C) -> -12V
- Q1 pad 3: -12V -> Net-(Q1-E)
- Q2 pad 1: /Sync -> Net-(D2-K)
- Q2 pad 2: Net-(Q1-C) -> Net-(Q1-E)
- R6 pad 2: Net-(Q1-C) -> Net-(Q1-E)
- TP2 pad 1: /Sync -> Net-(D2-K)
- U1 pad 3: /Sync -> Net-(D2-K)
- U2 pad 1: /Sync -> Net-(D2-K)
Routing:
- net Net-(D2-K): track 0.00 -> 63.3 mm, vias 0 -> 1
- net /Sync: track 76.2 -> 44.5 mm
- net +12V: track 287.1 -> 315.3 mm, vias 3 -> 2
- net Net-(C8-Pad1): track 0.00 -> 27.6 mm, vias 0 -> 1
- net Net-(Q1-E): track 0.00 -> 20.5 mm
- net Net-(Q1-C): track 20.2 -> 0.00 mm
- net /Fine_oct_in: track 38.4 -> 57.0 mm, vias 0 -> 1
- net /Saw: track 57.9 -> 39.7 mm, vias 1 -> 0
- net Net-(Q4-B): track 0.00 -> 15.2 mm
- net -12V: track 253.8 -> 243.2 mm, vias 4 -> 3
- net GND: track 0.00 -> 9.10 mm
- net Net-(D3-K): track 45.4 -> 54.1 mm
- net Net-(U4A-+): track 22.8 -> 16.6 mm
- net /octave: track 29.9 -> 35.5 mm, vias 0 -> 1
- net Net-(Q3-C): track 0.00 -> 4.47 mm
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Other:
- board text added: "1"
- board text added: "2"
- board text added: "3"
- board text added: "4"
- board text added: "5V"
- board text added: "CD40106 VCO 2.0 Bleep Sound 2025"
- board text removed: "CD40106 VCO 1.0 Bleep Sound 2023"
