File: fabrication/front/CD40106_VCO.kicad_pcb (KiCad board)
At the start: 2 copper layers, 50 x 128.5 mm, 5 parts

Commit message: V2.0
Parts:
- moved G*** 89.0 mm to (221.5, 147.0)
- moved H3 89.0 mm to (184.5, 30.5)
- moved H4 89.0 mm to (219.5, 30.5)
- moved H5 89.0 mm to (219.5, 153.0)
- moved H6 89.0 mm to (184.5, 153.0)
Other:
- board text added: "CD40106 VCO 2.0 Bleep Sound 2025"
- board text added: "Front panel"
- board text removed: "CD40106 VCO 1.0 Bleep Sound 2023"
- board text removed: "Front"
- board text removed: "MS-20 VCF Face plate V1.0 BleepSound 2022"
