File: fabrication/jackboard/CD40106_VCO.kicad_pcb (KiCad board)
At the start: 2 copper layers, 50 x 73.2 mm, 20 parts, among them J1 FM, J10 Square, J13 Sine, J15 Tri, J2 CV, J3 Sync, J4 PWM_CV, J6 Conn_Jack, J8 Conn_Jack, J9 Saw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

Commit message: V2.0
Parts:
- removed D1: 1N4148, Diode_THT:D_DO-35_SOD27_P7.62mm_Horizontal
- added C1: 470pF, Capacitor_THT:C_Disc_D7.0mm_W2.5mm_P5.00mm, F.Cu at (157.2, 113.1)
- added R41: 1k, Resistor_THT:R_Axial_DIN0207_L6.3mm_D2.5mm_P10.16mm_Horizontal, F.Cu at (142.0, 112.8)
- FM_LVL1: value 1M -> B1M
- Fine1: value 10k -> B10k
- PWM1: value 100k -> B100k
- PWM_CV_LVL1: value 250k -> B250k
Connections:
- J10 pad T: /Square out -> Net-(J10-PadT)
Routing:
- net /Square out: track 69.8 -> 33.1 mm
- net Net-(J10-PadT): track 0.00 -> 36.5 mm
- net Net-(C1-Pad1): track 16.2 -> 18.4 mm
- net GND: vias 25 -> 26
Other:
- board text added: "CD40106 VCO 2.0 Bleep Sound 2025"
- board text removed: "CD40106 VCO 1.0 Bleep Sound 2023"
