File: kicad-global/Power.kicad_sch (KiCad schematic)
At the start: 21 parts, among them J6 Power Input, U1 TL074, U2 40106, U3 LM13700, U4 TL074, U6 TL074

Commit message: finished v1 of module
Parts:
- removed C11, C12: 100n, Capacitor_THT:C_Disc_D7.0mm_W2.5mm_P5.00mm, symbol Device:C_Small
- removed D2: LED-12V, LED_THT:LED_D4.0mm, symbol Device:LED
- removed R19: 2.2k, Resistor_THT:R_Axial_DIN0207_L6.3mm_D2.5mm_P10.16mm_Horizontal, symbol Device:R
- removed U6: TL074, Package_DIP:DIP-14_W7.62mm_Socket, symbol Amplifier_Operational:TL074
- added C18, C19, C20, C21: 100nF, Capacitor_THT:C_Disc_D7.0mm_W2.5mm_P5.00mm, symbol Device:C_Small
- added U5: TL072, Package_DIP:DIP-8_W7.62mm_Socket, symbol Amplifier_Operational:TL072
- added unit 3 of U7
- C10: renamed from C4; value 10u -> 10uF
- C11: renamed from C5; value 10u -> 10uF
- C12: renamed from C6; value 100n -> 100nF
- C13: renamed from C7; value 100n -> 100nF
- C14: renamed from C8; value 100n -> 100nF
- C15: renamed from C9; value 100n -> 100nF
- C16: renamed from C15; value 100n -> 100nF
- C17: renamed from C16; value 100n -> 100nF
- C22: renamed from C10; value 100n -> 100nF
- FB1, FB2: footprint Inductor_THT:L_Axial_L9.5mm_D4.0mm_P12.70mm_Horizontal_Fastron_SMCC -> Inductor_THT:L_Axial_L7.0mm_D3.3mm_P10.16mm_Horizontal_Fastron_MICC; Comments (none) -> Ferrite beads (or inductance)
- U2: value 40106 -> CD40106; footprint (none) -> Package_DIP:DIP-14_W7.62mm_LongPads; manf (none) -> Nexperia; manf# (none) -> CD40106BE
- U6: renamed from U3; manf (none) -> Texas Instrument; manf# (none) -> LM13700MX/NOPB
- renumbered J6 to J16, U4 to U7
Connections:
- net +12V: now also C18.1, C20.1, U5.8 (V+), U7.8 (V+)
- net -12V: now also C19.2, C21.2, U5.4 (V-), U7.4 (V-)
- net GND: now also C18.2, C19.1, C20.2, C21.1
Other:
- moved on the sheet: C22, U1E, U2G, U6E, U7E

Commit message: doc + fab files for V1.0
Other:
- company: (none) -> Bleep Sound
- title: (none) -> CD40106 VCO
Changed lines of the file:
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@@
 (kicad_sch (version 20230121) (generator eeschema)
   (paper "A4")
+  (title_block
+    (title "CD40106 VCO")
+    (date "2023-12-10")
+    (rev "1.0")
+    (company "Bleep Sound")
+  )
   (junction (at 111.76 123.19) (diameter 0) (color 0 0 0 0)
   )

Commit message: First proto fix
Parts:
- removed FB1, FB2: 10R, Inductor_THT:L_Axial_L7.0mm_D3.3mm_P10.16mm_Horizontal_Fastron_MICC, symbol Device:Ferrite_Bead_Small
- added D6, D8: 1N5819, Diode_THT:D_DO-41_SOD81_P10.16mm_Horizontal, symbol Diode:1N5819
- renumbered U5 to U4, U7 to U5
Connections:
- net +12V: now also D6.1 (K)
- net -12V: now also D8.2 (A)
- net at J16.1 (Pin_1), J16.2 (Pin_2): now also D8.1 (K)
- net at J16.10 (Pin_10), J16.9 (Pin_9): now also D6.2 (A)

Commit message: V2.0
Parts:
- C10, C11: Links (none) -> https://www.taydaelectronics.com/capacitors/electrolytic-ca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
- C12, C13, C14, C15, C16, C17, C18, C19, C20, C21, C22: Links (none) -> https://www.taydaelectronics.com/capacitors/monolithic-cera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
- D6, D8: Links (none) -> https://www.taydaelectronics.com/1n5819-schottky-barrier-di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
- J16: Links (none) -> https://www.thonk.co.uk/shop/eurorack-diy-essentials/
- U1, U7: Links (none) -> https://www.thonk.co.uk/shop/eurorack-diy-essentials/; manf (none) -> Texas Instrument; manf# (none) -> TL074CN
- U2: Links (none) -> https://eu.mouser.com/ProductDetail/Texas-Instruments/CD401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
- U4, U5: Links (none) -> https://eu.mouser.com/ProductDetail/Texas-Instruments/TL072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; manf (none) -> Texas Instrument; manf# (none) -> TL072IP
- U6: Links (none) -> https://eu.mouser.com/c/semiconductors/amplifier-ics/transc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
