File: kicad-global/octave_switch.kicad_sch (KiCad schematic)
At the start: 21 parts, among them SW1 Octave select switch, U4 TL074, U5 LM336BZ-5.0

Commit message: finished v1 of module
Parts:
- removed U4: TL074, Package_DIP:DIP-14_W7.62mm_Socket, symbol Amplifier_Operational:TL074
- added J11: Conn_01x04, Connector_PinHeader_2.54mm:PinHeader_1x04_P2.54mm_Vertical, symbol Connector_Generic:Conn_01x04
- added J12: Conn_01x04, Connector_PinSocket_2.54mm:PinSocket_1x04_P2.54mm_Vertical, symbol Connector_Generic:Conn_01x04
- added U4, U5: TL072, Package_DIP:DIP-8_W7.62mm_Socket, symbol Amplifier_Operational:TL072
- C14: value 100n -> 100nF
- C14: value 1n -> 1nF
- Coarse: footprint Synth:Pot-bourns-alpha -> Kicad-perso:Pot-bourns-alpha
- SW1: footprint (none) -> Kicad-perso:CK1055; manf (none) -> Lorlin; manf# (none) -> CK1055
- TP3: renamed from TP1; footprint (none) -> TestPoint:TestPoint_Plated_Hole_D2.0mm
- renumbered U5 to U3
Connections:
- net 2V: now also SW1.3; no longer SW1.4
- net 3V: now also SW1.4; no longer SW1.3
- net 4V: now also SW1.5; no longer SW1.2
- net 5v: now also SW1.6, J11.2 (Pin_2), J12.2 (Pin_2), U4.1; no longer SW1.1
- net Fine: now also U5.6 (-), U5.7
- net GND: now also C14.1, SW1.1, J11.4 (Pin_4), J12.4 (Pin_4); no longer C14.2, SW1.6
- net Octave: now also U4.6 (-), U4.7
- net at C14.2, Coarse.2: now also U5.5 (+)
- net at R7.1, R7.2: now also U4.2 (-)
- net at Coarse.1: now also U5.1, U5.2 (-)
- net at R7.1: now also U4.3 (+)
- net 1V renamed Fine_oct_in
- net Fine_oct_in: now also SW1.2, J11.3 (Pin_3), J12.3 (Pin_3), U5.3 (+); no longer SW1.5
- new net A: C14.2, J11.1 (Pin_1), J12.1 (Pin_1), SW1.A, U4.5 (+)
Other:
- note added: "Five octave switch"
- note added: "One octave fine adjust pot"
- note added: "Taken from MFOS, designed by Ray Wilson"
- note removed: "One octave adjust pot"
- note removed: "Tl072 instead ?"

Commit message: doc + fab files for V1.0
Other:
- company: (none) -> Bleep Sound
- title: (none) -> CD40106 VCO
Changed lines of the file:
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@@
 (kicad_sch (version 20230121) (generator eeschema)
   (paper "A4")
+  (title_block
+    (title "CD40106 VCO")
+    (date "2023-12-10")
+    (rev "1.0")
+    (company "Bleep Sound")
+  )
   (junction (at 119.38 50.8) (diameter 0) (color 0 0 0 0)
   )

Commit message: First proto fix
Parts:
- Fine1: renamed from Coarse; value 10k -> B10k
- R24: renamed from R7; value 9k53 -> 9k1
- U3: value LM336BZ-5.0 -> LM336-2.5; manf# LM336BZ-5.0/NOPB -> LM336-2.5
- lvl_Trim2: renamed from lvl_Trim; value 1k -> 2k
- renumbered C14 to C4, C14 to C5, C14 to C6, C14 to C7, R7 to R16, R7 to R17, R7 to R18, R7 to R19, R5 to R20, R7 to R21, R4 to R22, R3 to R23, R2 to R25, R1 to R26

Commit message: V2.0
Parts:
- C4, C5, C6, C7: Links (none) -> https://www.taydaelectronics.com/capacitors/monolithic-cera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
- Fine1: Links (none) -> https://www.thonk.co.uk/shop/alpha-9mm-pots/
- R16, R17, R18, R19, R20, R21, R22, R23, R24, R25, R26: Links (none) -> https://www.taydaelectronics.com/resistors/1-4w-metal-film-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
- SW1: Comments (none) -> Cut the shaft to required length; Links (none) -> https://uk.rs-online.com/web/p/rotary-switches/8660278?sear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
- U3: Links (none) -> https://uk.rs-online.com/web/p/voltage-references/5335799P?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
- U4, U5: Links (none) -> https://eu.mouser.com/ProductDetail/Texas-Instruments/TL072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; manf (none) -> Texas Instrument; manf# (none) -> TL072IP
- lvl_Trim2: footprint Potentiometer_THT:Potentiometer_Bourns_3386C_Horizontal -> Potentiometer_THT:Potentiometer_Bourns_3296W_Vertical; Links (none) -> Trimmer potentiometer, 25 turn series 3296W
